File: 0032_Servo_Drive_PCA9685.kicad_sch (KiCad schematic)
At the start: 14 parts, among them J1 Screw_Terminal_01x15, J2 Screw_Terminal_01x15, U1 PCA9685PW

Commit message: Add files via upload
Parts:
- removed J1, J2: Screw_Terminal_01x15, symbol Connector:Screw_Terminal_01x15
- removed R3, R4, R5, R6, R7: 0r, symbol Device:R
- removed RN3: 10k, symbol Device:R_Pack06
- added D1: LED, LED_SMD:LED_0603_1608Metric, symbol Device:LED
- added J1, J10, J2, J3, J4, J5, J6, J7, J8, J9: Screw_Terminal_01x03, Connector_PinSocket_2.54mm:PinSocket_1x03_P2.54mm_Vertical, symbol Connector:Screw_Terminal_01x03
- added JP1, JP2, JP3, JP4, JP5: SolderJumper_2_Open, Jumper:SolderJumper-2_P1.3mm_Open_RoundedPad1.0x1.5mm, symbol Jumper:SolderJumper_2_Open
- added JP6: ESolderJumper_2_Open, Jumper:SolderJumper-2_P1.3mm_Open_RoundedPad1.0x1.5mm, symbol Jumper:SolderJumper_2_Open
- added RN3, RN4: R_Pack04, Resistor_SMD:R_Array_Concave_4x0402, symbol Device:R_Pack04
- added U2: ~, Moduler_:pin_header_5-3, symbol moduler_pin:air
- C1: footprint (none) -> Capacitor_SMD:C_0603_1608Metric
- R1: footprint (none) -> Resistor_SMD:R_0603_1608Metric
- R2: value 0r -> R; footprint (none) -> Resistor_SMD:R_0603_1608Metric
Connections:
- net A0: now also JP1.2 (B), RN3.7 (R2.2); no longer R2.2
- net A1: now also JP2.2 (B), RN3.6 (R3.2)
- net A2: now also JP3.2 (B), RN3.5 (R4.2)
- net A3: now also JP4.2 (B), RN4.8 (R1.2)
- net A4: now also JP5.2 (B), RN4.7 (R2.2)
- net A5: now also JP6.2 (B), RN4.6 (R3.2)
- net GND: now also D1.1 (K), J1.3 (Pin_3), J10.3 (Pin_3), J2.3 (Pin_3), J3.3 (Pin_3), J4.3 (Pin_3), J5.3 (Pin_3), J6.3 (Pin_3), J7.3 (Pin_3), J8.3 (Pin_3), J9.3 (Pin_3), RN3.1 (R1.1), RN3.2 (R2.1), RN3.3 (R3.1), RN3.4 (R4.1), RN4.1 (R1.1), RN4.2 (R2.1), RN4.3 (R3.1), RN4.4 (R4.1), U2.9
- net SCL: now also U2.5
- net SDA: now also U2.6
- net at RN2.10 (R1.2): now also J6.1 (Pin_1)
- net at RN2.6 (R5.2): now also J10.1 (Pin_1)
- net at RN2.7 (R4.2): now also J9.1 (Pin_1)
- net at RN2.8 (R3.2): now also J8.1 (Pin_1)
- net at RN2.9 (R2.2): now also J7.1 (Pin_1)
- net at RN1.10 (R1.2): now also J1.1 (Pin_1)
- net at RN1.7 (R4.2): now also J4.1 (Pin_1)
- net at RN1.6 (R5.2): now also J5.1 (Pin_1)
- net at RN1.9 (R2.2): now also J2.1 (Pin_1)
- net at RN1.8 (R3.2): now also J3.1 (Pin_1)
- net OE: now reaches R1.1, U1.23 (~{OE})
- net OE: now also U2.12
- net VCC renamed +3V3
- net +3V3: now also J1.2 (Pin_2), J10.2 (Pin_2), J2.2 (Pin_2), J3.2 (Pin_2), J4.2 (Pin_2), J5.2 (Pin_2), J6.2 (Pin_2), J7.2 (Pin_2), J8.2 (Pin_2), J9.2 (Pin_2), JP1.1 (A), JP2.1 (A), JP3.1 (A), JP4.1 (A), JP5.1 (A), JP6.1 (A), U2.8
- new net: D1.2 (A), R2.2
- no-connect marks 6 -> 21
Other:
- note added: "AIR PIN"
- note added: "JUMPER"
- note added: "PIN HEADER"
- note added: "SENSOR"
- moved on the sheet: C1, R1, RN1, RN2, U1
